File: MU-TH-UR pad/KiCad/MU-TH-UR pad/MU-TH-UR pad.kicad_pcb (KiCad board)
At the start: 2 copper layers, 186.4 x 62.7 mm, 43 parts, among them J1 OLED_DISPLAY, SW1 RotaryEncoder_Switch, SW2 SW_Push_45deg, SW3 SW_Push_45deg, SW4 SW_Push_45deg, SW5 SW_Push_45deg, U3 RP2040-Zero

Commit message: JLCPCB Gerbers
Other:
- board text removed: "WayWayWay"
